Commit message: added gazebo launch file

File: src/franky_description/URDF/franky.urdf.xacro (robot description, xacro)
@@ -1,14 +1,29 @@
 <?xml version="1.0"?>
 <robot xmlns:xacro="http://www.ros.org/wiki/xacro" name="franky">
+    <!-- Include Gazebo Parameters -->
+    <xacro:include filename="$(find franky_description)/URDF/franky_gazebo.xacro" />
     <link name="base_footprint"/>
     <link name="base_link">
+        <inertial>
+            <origin xyz="0 0 0.04" rpy="0.0 0.25 0.3" />
+            <mass value="8.2573504e-01"/>
+            <inertia ixx="2.2124416e-02" ixy="-1.2294101e-04" ixz="3.4938785e-04"
+                iyy="2.1193702e-02" iyz="-5.0120904e-05"
+                izz="2.0064271e-02" />
+        </inertial>
         <visual>
             <geometry>
                 <mesh filename="package://franky_description/meshes/base_link.STL"/>
             </geometry>
-            <material name="base_material">
+            <material name="white">
                 <color rgba="1.0 1.0 1.0 1.0"/>
             </material>
         </visual>
+        <collision>
+            <origin xyz="0 0 0" rpy="0 0 0" />
+            <geometry>
+                <mesh filename="package://bumperbot_description/meshes/base_link.STL" />
+            </geometry>
+        </collision>
     </link>
     <joint name="base_joint" type="fixed">
@@ -18,4 +33,11 @@
     </joint>
     <link name="wheel_right_link">
+        <inertial>
+            <origin xyz="0 -0.014 0" rpy="0 0 0" />
+            <mass value="0.0530086090966721" />
+            <inertia ixx="1.88176298336665E-05" ixy="-4.8444933029987E-10" ixz="1.88163708851143E-08"
+               iyy="3.11510738647764E-05" iyz="-6.93560663069607E-11"
+               izz="1.8801969558182E-05" />
+        </inertial>
         <visual>
             <origin xyz="0 0 0" rpy="1.57 0 0"/>
@@ -23,8 +45,14 @@
                 <mesh filename="package://franky_description/meshes/wheel_right_link.STL"/>
             </geometry>
-            <material name="wheel_material">
+            <material name="black">
                 <color rgba="0.2 0.2 0.2 1.0"/>
             </material>
         </visual>
+        <collision>
+            <origin xyz="0 -0.015 0" rpy="1.57 0 0" />
+            <geometry>
+                <sphere radius="0.033"/>
+            </geometry>
+        </collision>
     </link>
     <joint name="wheel_right_joint" type="continuous">
@@ -35,4 +63,11 @@
     </joint>
     <link name="wheel_left_link">
+        <inertial>
+            <origin xyz="0 0.014 0" rpy="0 0 0" />
+            <mass value="0.0530086043217644" />
+            <inertia ixx="1.8792911368909E-05"  ixy="3.31256392204584E-10" ixz="-1.14082001662767E-08"
+               iyy="3.11510738759073E-05" iyz="-3.60499245082192E-10"
+               izz="1.88266886146847E-05" />
+        </inertial>
         <visual>
             <origin xyz="0 0 0" rpy="-1.57 0 0"/>
@@ -40,8 +75,14 @@
                 <mesh filename="package://franky_description/meshes/wheel_left_link.STL"/>
             </geometry>
-            <material name="wheel_material">
+            <material name="black">
                 <color rgba="0.2 0.2 0.2 1.0"/>
             </material>
         </visual>
+        <collision>
+            <origin xyz="0 0.015 0" rpy="-1.57 0 0" />
+            <geometry>
+                <sphere radius="0.033"/>
+            </geometry>
+        </collision>
     </link>
     <joint name="wheel_left_joint" type="continuous">
@@ -52,4 +93,11 @@
     </joint>
     <link name="caster_front_link">
+        <inertial>
+            <origin xyz="3.89968128948481E-07 2.40073004698083E-07 0.00219173397061506" rpy="0 0 0" />
+            <mass value="1.44379265037903E-06" />
+            <inertia ixx="7.23075276010246E-11" ixy="-6.10956883467859E-16" ixz="2.22849693525031E-15"
+               iyy="3.8713793085917E-11"  iyz="2.93909858781952E-15"
+               izz="1.00967486676306E-10" />
+        </inertial>
         <visual>
             <origin xyz="0 0 0" rpy="0 0 0"/>
@@ -61,4 +109,10 @@
             </material>
         </visual>
+        <collision>
+            <origin xyz="0 0 0" rpy="0 0 0" />
+            <geometry>
+                <sphere radius="0.005"/>
+            </geometry>
+        </collision>
     </link>
     <joint name="caster_front_joint" type="fixed">
@@ -68,4 +122,11 @@
     </joint>
     <link name="caster_rear_link">
+        <inertial>
+            <origin xyz="3.8996812895542E-07 2.40073004698083E-07 0.00219173397061509" rpy="0 0 0" />
+            <mass value="1.44379265037902E-06" />
+            <inertia ixx="7.23075276010246E-11" ixy="-6.10956872363424E-16" ixz="2.22849693527207E-15"
+               iyy="3.87137930859167E-11" iyz="2.939098587861E-15"
+               izz="1.00967486676306E-10" />
+        </inertial>
         <visual>
             <origin xyz="0 0 0" rpy="0 0 0"/>
@@ -77,4 +138,10 @@
             </material>
         </visual>
+        <collision>
+            <origin xyz="0 0 0" rpy="0 0 0" />
+            <geometry>
+                <sphere radius="0.005"/>
+            </geometry>
+        </collision>
     </link>
     <joint name="caster_rear_joint" type="fixed">
@@ -83,3 +150,19 @@
         <origin rpy="0 0 0" xyz="-0.04755 0 -0.0275"/>
     </joint>
+<!--    <link name="can_link">
+        <visual>
+            <origin xyz="-0.03 0.033 0" rpy="1.57 0 0"/>
+            <geometry>
+                <mesh filename="package://franky_description/meshes/can.STL"/>
+            </geometry>
+            <material name="red">
+                <color rgba="1.0 0.0 0.0 1.0"/>
+            </material>
+        </visual>
+    </link>
+    <joint name="can_joint" type="fixed">
+        <parent link="base_link"/>
+        <child link="can_link"/>
+        <origin rpy="0 0 0" xyz="0 0 0.078"/>
+    </joint>"""" -->
 </robot>

Commit message: added controller plugin

File: src/franky_description/URDF/franky.urdf.xacro (robot description, xacro)
@@ -1,6 +1,9 @@
 <?xml version="1.0"?>
 <robot xmlns:xacro="http://www.ros.org/wiki/xacro" name="franky">
+    <xacro:arg name="is_ignition" default="true"/>
     <!-- Include Gazebo Parameters -->
     <xacro:include filename="$(find franky_description)/URDF/franky_gazebo.xacro" />
+    <!-- Include ros2_control -->
+    <xacro:include filename="$(find franky_description)/URDF/franky_ros2_control.xacro" />
     <link name="base_footprint"/>
     <link name="base_link">
@@ -165,4 +168,5 @@
         <child link="can_link"/>
         <origin rpy="0 0 0" xyz="0 0 0.078"/>
-    </joint>"""" -->
+    </joint>
+-->
 </robot>

File: src/franky_description/URDF/franky_gazebo.xacro (robot description, xacro)
@@ -35,3 +35,15 @@
         <maxVel>0.1</maxVel>
     </gazebo>
+    <gazebo>
+        <xacro:if value="$(arg is_ignition)">
+            <plugin filename="ign_ros2_control-system" name="ign_ros2_control::IgnitionROS2ControlPlugin">
+                <parameters>$(find franky_controller)/config/franky_controllers.yaml</parameters>
+            </plugin>
+        </xacro:if>
+        <xacro:unless value="$(arg is_ignition)">
+            <plugin filename="gz_ros2_control-system" name="gz_ros2_control::GazeboSimROS2ControlPlugin">
+                <parameters>$(find franky_controller)/config/franky_controllers.yaml</parameters>
+            </plugin>
+        </xacro:unless>
+    </gazebo>
 </robot>

Commit message: added controller launch file

File: src/franky_description/URDF/franky.urdf.xacro (robot description, xacro)
@@ -26,5 +26,5 @@
             <origin xyz="0 0 0" rpy="0 0 0" />
             <geometry>
-                <mesh filename="package://bumperbot_description/meshes/base_link.STL" />
+                <mesh filename="package://franky_description/meshes/base_link.STL" />
             </geometry>
         </collision>

Commit message: updated inverse diff kinematics

File: src/franky_description/URDF/franky.urdf.xacro (robot description, xacro)
@@ -23,7 +23,7 @@
         </visual>
         <collision>
-            <origin xyz="0 0 0" rpy="0 0 0" />
+            <origin xyz="0 0 0.04" rpy="0 0 0" />
             <geometry>
-                <mesh filename="package://franky_description/meshes/base_link.STL" />
+                <box size="0.18 0.14 0.08" />
             </geometry>
         </collision>
