Commit message: integrated imu

File: franky_description/URDF/franky.urdf.xacro (robot description, xacro)
@@ -152,4 +152,34 @@
         <origin rpy="0 0 0" xyz="-0.04755 0 -0.0275"/>
     </joint>
+    <link name="imu_link">
+        <inertial>
+          <origin xyz="-0.00552433659106688 0.000168210391520346 0.000514000497342681" rpy="0 0 0" />
+          <mass value="0.000528415362211671" />
+          <inertia ixx="1.46176048428261E-08" ixy="1.40015117949421E-10" ixz="-1.99633872937403E-12"
+                   iyy="8.59662482954888E-09" iyz="7.52375112767959E-12"
+                   izz="2.30279421279312E-08" />
+        </inertial>
+        <visual>
+          <origin xyz="0 0 0" rpy="0 0 0" />
+          <geometry>
+            <mesh filename="package://bumperbot_description/meshes/imu_link.STL" />
+          </geometry>
+          <material name="">
+            <color rgba="0.792156862745098 0.819607843137255 0.933333333333333 1" />
+          </material>
+        </visual>
+        <collision>
+          <origin xyz="0 0 0" rpy="0 0 0" />
+          <geometry>
+            <mesh filename="package://bumperbot_description/meshes/imu_link.STL" />
+          </geometry>
+        </collision>
+    </link>
+    <joint name="imu_joint" type="fixed">
+        <origin xyz="0 0 0.0698986241758014" rpy="0 0 0" />
+        <parent link="base_link" />
+        <child link="imu_link" />
+        <axis xyz="0 0 0" />
+    </joint>
 <!--    <link name="can_link">
         <visual>

File: franky_description/URDF/franky_gazebo.xacro (robot description, xacro)
@@ -1,4 +1,5 @@
 <?xml version="1.0"?>
 <robot name="franky" xmlns:xacro="http://www.ros.org/wiki/xacro">
+    <!-- Wheels -->
     <gazebo reference="wheel_right_link">
         <mu1>100000000000000.0</mu1>
@@ -19,4 +20,5 @@
         <fdir1>1 0 0</fdir1>
     </gazebo>
+    <!-- Caster wheels -->
     <gazebo reference="caster_front_link">
         <mu1>0.1</mu1>
@@ -35,8 +37,61 @@
         <maxVel>0.1</maxVel>
     </gazebo>
+    <!-- IMU -->
+    <gazebo reference="imu_link">
+      <sensor name="imu" type="imu">
+          <always_on>true</always_on>
+          <update_rate>50</update_rate>
+          <gz_frame_id>imu_link</gz_frame_id>
+          <topic>imu</topic>
+          <imu>
+            <angular_velocity>
+              <x>
+                <noise type="gaussian">
+                  <mean>0.0</mean>
+                  <stddev>2e-4</stddev>
+                </noise>
+              </x>
+              <y>
+                <noise type="gaussian">
+                  <mean>0.0</mean>
+                  <stddev>2e-4</stddev>
+                </noise>
+              </y>
+              <z>
+                <noise type="gaussian">
+                  <mean>0.0</mean>
+                  <stddev>2e-4</stddev>
+                </noise>
+              </z>
+            </angular_velocity>
+            <linear_acceleration>
+              <x>
+                <noise type="gaussian">
+                  <mean>0.0</mean>
+                  <stddev>1.7e-2</stddev>
+                </noise>
+              </x>
+              <y>
+                <noise type="gaussian">
+                  <mean>0.0</mean>
+                  <stddev>1.7e-2</stddev>
+                </noise>
+              </y>
+              <z>
+                <noise type="gaussian">
+                  <mean>0.0</mean>
+                  <stddev>1.7e-2</stddev>
+                </noise>
+              </z>
+            </linear_acceleration>
+          </imu>
+      </sensor>
+    </gazebo>
     <gazebo>
         <plugin filename="gz_ros2_control-system" name="gz_ros2_control::GazeboSimROS2ControlPlugin">
             <parameters>$(find franky_controller)/config/franky_controllers.yaml</parameters>
         </plugin>
+        <plugin filename="gz-sim-imu-system" name="gz::sim::systems::Imu">
+        </plugin>
     </gazebo>
 </robot>

Commit message: added ekf and urdf lidar corrections

File: franky_description/URDF/franky.urdf.xacro (robot description, xacro)
@@ -163,5 +163,5 @@
           <origin xyz="0 0 0" rpy="0 0 0" />
           <geometry>
-            <mesh filename="package://bumperbot_description/meshes/imu_link.STL" />
+            <mesh filename="package://franky_description/meshes/imu_link.STL" />
           </geometry>
           <material name="">
@@ -172,5 +172,5 @@
           <origin xyz="0 0 0" rpy="0 0 0" />
           <geometry>
-            <mesh filename="package://bumperbot_description/meshes/imu_link.STL" />
+            <mesh filename="package://franky_description/meshes/imu_link.STL" />
           </geometry>
         </collision>
@@ -182,9 +182,16 @@
         <axis xyz="0 0 0" />
     </joint>
-<!--    <link name="can_link">
-        <visual>
-            <origin xyz="-0.03 0.033 0" rpy="1.57 0 0"/>
-            <geometry>
-                <mesh filename="package://franky_description/meshes/can.STL"/>
+    <link name="lidar_link">
+        <inertial>
+            <origin xyz="0 0 0" rpy="0 0 0" />
+            <mass value="0.2" />
+            <inertia ixx="0.0001" ixy="0.0" ixz="0.0"
+                     iyy="0.0001" iyz="0.0"
+                     izz="0.0001" />
+        </inertial>
+        <visual>
+            <origin xyz="0 0 0" rpy="0 0 0"/>
+            <geometry>
+                <mesh filename="package://franky_description/meshes/laser_link.STL"/>
             </geometry>
             <material name="red">
@@ -192,10 +199,15 @@
             </material>
         </visual>
-    </link>
-    <joint name="can_joint" type="fixed">
-        <parent link="base_link"/>
-        <child link="can_link"/>
-        <origin rpy="0 0 0" xyz="0 0 0.078"/>
-    </joint>
--->
+        <collision>
+            <origin xyz="0 0 0" rpy="0 0 0"/>
+            <geometry>
+                <mesh filename="package://franky_description/meshes/laser_link.STL"/>
+            </geometry>
+        </collision>
+    </link>
+    <joint name="lidar_joint" type="fixed">
+        <parent link="base_link"/>
+        <child link="lidar_link"/>
+        <origin rpy="0 0 0" xyz="0.0 0.0 0.11"/>
+    </joint>
 </robot>

Commit message: priority node

File: franky_description/URDF/franky.urdf.xacro (robot description, xacro)
@@ -165,6 +165,6 @@
             <mesh filename="package://franky_description/meshes/imu_link.STL" />
           </geometry>
-          <material name="">
-            <color rgba="0.792156862745098 0.819607843137255 0.933333333333333 1" />
+          <material name="blue">
+            <color rgba="0.0 0.0 1 1" />
           </material>
         </visual>
@@ -182,32 +182,33 @@
         <axis xyz="0 0 0" />
     </joint>
-    <link name="lidar_link">
-        <inertial>
-            <origin xyz="0 0 0" rpy="0 0 0" />
-            <mass value="0.2" />
-            <inertia ixx="0.0001" ixy="0.0" ixz="0.0"
-                     iyy="0.0001" iyz="0.0"
-                     izz="0.0001" />
-        </inertial>
-        <visual>
-            <origin xyz="0 0 0" rpy="0 0 0"/>
-            <geometry>
-                <mesh filename="package://franky_description/meshes/laser_link.STL"/>
-            </geometry>
-            <material name="red">
-                <color rgba="1.0 0.0 0.0 1.0"/>
-            </material>
-        </visual>
-        <collision>
-            <origin xyz="0 0 0" rpy="0 0 0"/>
-            <geometry>
-                <mesh filename="package://franky_description/meshes/laser_link.STL"/>
-            </geometry>
-        </collision>
-    </link>
-    <joint name="lidar_joint" type="fixed">
-        <parent link="base_link"/>
-        <child link="lidar_link"/>
-        <origin rpy="0 0 0" xyz="0.0 0.0 0.11"/>
+    <link name="laser_link">
+        <inertial>
+          <origin xyz="-0.011945780406062 -0.000381929217680526 -0.0170649378129477" rpy="0 0 0" />
+          <mass value="0.073084435549317" />
+          <inertia ixx="1.96074931730795E-05" ixy="-3.62091076640009E-07" ixz="4.28230084046735E-07"
+                   iyy="2.40983835136327E-05" iyz="1.50180909250652E-08"
+                   izz="4.14184164228595E-05" />
+        </inertial>
+        <visual>
+          <origin xyz="0 0 0" rpy="0 0 0" />
+          <geometry>
+            <mesh filename="package://franky_description/meshes/laser_link.STL" />
+          </geometry>
+          <material name="Red">
+            <color rgba="0.0 0.0 1 1"/>
+          </material>
+        </visual>
+        <collision>
+          <origin xyz="0 0 0" rpy="0 0 0" />
+          <geometry>
+            <mesh filename="package://franky_description/meshes/laser_link.STL" />
+          </geometry>
+        </collision>
+    </link>
+    <joint name="laser_joint" type="fixed">
+        <origin xyz="-0.0050526 -0.0023221 0.1208" rpy="0 0 3.14" />
+        <parent link="base_link" />
+        <child link="laser_link" />
+        <axis xyz="0 0 0" />
     </joint>
 </robot>

File: franky_description/URDF/franky_gazebo.xacro (robot description, xacro)
@@ -88,10 +88,51 @@
       </sensor>
     </gazebo>
+    <!-- 2D Laser Sensor -->
+    <gazebo reference="laser_link">
+      <sensor name="lidar" type="gpu_lidar">
+        <always_on>true</always_on>
+        <visualize>true</visualize>
+        <topic>scan</topic>
+        <update_rate>5</update_rate>
+        <gz_frame_id>laser_link</gz_frame_id>
+        <lidar>
+          <scan>
+            <horizontal>
+              <samples>360</samples>
+              <resolution>1.00000</resolution>
+              <min_angle>0.000000</min_angle>
+              <max_angle>6.280000</max_angle>
+            </horizontal>
+          </scan>
+          <range>
+            <min>0.120000</min>
+            <max>12.0</max>
+            <resolution>0.01</resolution>
+          </range>
+          <noise>
+            <type>gaussian</type>
+            <mean>0.0</mean>
+            <stddev>0.01</stddev>
+          </noise>
+        </lidar>
+      </sensor>
+    </gazebo>
     <gazebo>
-        <plugin filename="gz_ros2_control-system" name="gz_ros2_control::GazeboSimROS2ControlPlugin">
-            <parameters>$(find franky_controller)/config/franky_controllers.yaml</parameters>
-        </plugin>
-        <plugin filename="gz-sim-imu-system" name="gz::sim::systems::Imu">
-        </plugin>
+      <plugin
+        filename="gz-sim-sensors-system"
+        name="gz::sim::systems::Sensors">
+        <render_engine>ogre2</render_engine>
+      </plugin>
+      <plugin
+        filename="gz-sim-imu-system"
+        name="gz::sim::systems::Imu">
+      </plugin>
+      <plugin
+        filename="gz_ros2_control-system"
+        name="gz_ros2_control::GazeboSimROS2ControlPlugin">
+        <parameters>
+          $(find franky_controller)/config/franky_controllers.yaml
+        </parameters>
+      </plugin>
     </gazebo>
 </robot>
